File: 65c02-Computer/reset.sch (KiCad schematic (older format))
At the start: 9 parts, among them SW1 SW_Push, U3 74LS04, U5 LM555

Commit message: Create v2
Parts:
- added J4: Conn_01x02, Connector_PinHeader_2.54mm:PinHeader_1x02_P2.54mm_Vertical, symbol Connector_Generic:Conn_01x02
- C2: renamed from C1; footprint Capacitor_SMD:C_0603_1608Metric -> Capacitor_THT:C_Disc_D3.8mm_W2.6mm_P2.50mm
- C3: renamed from C2; footprint Capacitor_SMD:C_0603_1608Metric -> Capacitor_THT:C_Disc_D3.8mm_W2.6mm_P2.50mm
- C4: renamed from C3; footprint Capacitor_SMD:CP_Elec_4x3 -> Capacitor_THT:CP_Radial_D8.0mm_P5.00mm
- R5: renamed from R4; footprint Resistor_SMD:R_0603_1608Metric -> Resistor_THT:R_Axial_DIN0207_L6.3mm_D2.5mm_P10.16mm_Horizontal
- R6: renamed from R5; footprint Resistor_SMD:R_0603_1608Metric -> Resistor_THT:R_Axial_DIN0207_L6.3mm_D2.5mm_P10.16mm_Horizontal
- R7: renamed from R6; footprint Resistor_SMD:R_0603_1608Metric -> Resistor_THT:R_Axial_DIN0207_L6.3mm_D2.5mm_P10.16mm_Horizontal
- SW1: footprint Button_Switch_SMD:SW_SPST_B3S-1000 -> Button_Switch_THT:SW_PUSH_6mm_H4.3mm
- renumbered U5 to U7, U3 to U8
Connections:
- net GND: now also J4.2 (Pin_2)
- net at C2.1, R5.2, SW1.2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: now also J4.1 (Pin_1)
Changed lines of the file:
@@
 $EndDescr
 $Comp
-L Timer:LM555 U5
+L Timer:LM555 U7
 U 1 1 5DBF360E
 P 5300 3850
-F 0 "U5" H 5300 4431 50  0000 C CNN
+F 0 "U7" H 5300 4431 50  0000 C CNN
 F 1 "LM555" H 5300 4340 50  0000 C CNN
 F 2 "Package_DIP:DIP-8_W7.62mm" H 5300 3850 50  0001 C CNN
@@
 $EndComp
 $Comp
-L device:C C2
+L device:C C3
 U 1 1 5DBF406D
 P 5550 3200
-F 0 "C2" H 5665 3246 50  0000 L CNN
+F 0 "C3" H 5665 3246 50  0000 L CNN
 F 1 "C" H 5665 3155 50  0000 L CNN
-F 2 "Capacitor_SMD:C_0603_1608Metric" H 5588 3050 50  0001 C CNN
+F 2 "Capacitor_THT:C_Disc_D3.8mm_W2.6mm_P2.50mm" H 5588 3050 50  0001 C CNN
 F 3 "~" H 5550 3200 50  0001 C CNN
 	1    5550 3200
@@
 $EndComp
 $Comp
-L power:GND #PWR015
+L power:GND #PWR036
 U 1 1 5DBF4F6E
 P 5550 3350
-F 0 "#PWR015" H 5550 3100 50  0001 C CNN
+F 0 "#PWR036" H 5550 3100 50  0001 C CNN
 F 1 "GND" H 5650 3250 50  0000 C CNN
 F 2 "" H 5550 3350 50  0001 C CNN
@@
 $EndComp
 $Comp
-L power:+5V #PWR014
+L power:+5V #PWR035
 U 1 1 5DBF5A36
 P 5550 2950
-F 0 "#PWR014" H 5550 2800 50  0001 C CNN
+F 0 "#PWR035" H 5550 2800 50  0001 C CNN
 F 1 "+5V" H 5565 3123 50  0000 C CNN
 F 2 "" H 5550 2950 50  0001 C CNN
@@
 Connection ~ 5300 3000
 $Comp
-L 74xx:74LS04 U3
+L 74xx:74LS04 U8
 U 1 1 5DBF6CEB
 P 6300 3650
-F 0 "U3" H 6300 3967 50  0000 C CNN
+F 0 "U8" H 6300 3967 50  0000 C CNN
 F 1 "74LS04" H 6300 3876 50  0000 C CNN
 F 2 "Package_DIP:DIP-14_W7.62mm" H 6300 3650 50  0001 C CNN
@@
 $EndComp
 $Comp
-L device:C C1
+L device:C C2
 U 1 1 5DBF8323
 P 4350 3850
-F 0 "C1" H 4465 3896 50  0000 L CNN
+F 0 "C2" H 4465 3896 50  0000 L CNN
 F 1 "100n" H 4465 3805 50  0000 L CNN
-F 2 "Capacitor_SMD:C_0603_1608Metric" H 4388 3700 50  0001 C CNN
+F 2 "Capacitor_THT:C_Disc_D3.8mm_W2.6mm_P2.50mm" H 4388 3700 50  0001 C CNN
 F 3 "~" H 4350 3850 50  0001 C CNN
 	1    4350 3850
@@
 $EndComp
 $Comp
-L device:CP1 C3
+L device:CP1 C4
 U 1 1 5DBFB427
 P 5900 4300
-F 0 "C3" H 6015 4346 50  0000 L CNN
+F 0 "C4" H 6015 4346 50  0000 L CNN
 F 1 "10u" H 6015 4255 50  0000 L CNN
-F 2 "Capacitor_SMD:CP_Elec_4x3" H 5900 4300 50  0001 C CNN
+F 2 "Capacitor_THT:CP_Radial_D8.0mm_P5.00mm" H 5900 4300 50  0001 C CNN
 F 3 "~" H 5900 4300 50  0001 C CNN
 	1    5900 4300
@@
 $EndComp
 $Comp
-L device:R R4
+L device:R R5
 U 1 1 5DBFC478
 P 4350 3450
-F 0 "R4" H 4420 3496 50  0000 L CNN
+F 0 "R5" H 4420 3496 50  0000 L CNN
 F 1 "1M" H 4420 3405 50  0000 L CNN
-F 2 "Resistor_SMD:R_0603_1608Metric" V 4280 3450 50  0001 C CNN
+F 2 "Resistor_THT:R_Axial_DIN0207_L6.3mm_D2.5mm_P10.16mm_Horizontal" V 4280 3450 50  0001 C CNN
 F 3 "~" H 4350 3450 50  0001 C CNN
 	1    4350 3450
@@
 $EndComp
 $Comp
-L device:R R5
+L device:R R6
 U 1 1 5DBFD8CE
 P 5900 3200
-F 0 "R5" H 5970 3246 50  0000 L CNN
+F 0 "R6" H 5970 3246 50  0000 L CNN
 F 1 "30k" H 5970 3155 50  0000 L CNN
-F 2 "Resistor_SMD:R_0603_1608Metric" V 5830 3200 50  0001 C CNN
+F 2 "Resistor_THT:R_Axial_DIN0207_L6.3mm_D2.5mm_P10.16mm_Horizontal" V 5830 3200 50  0001 C CNN
 F 3 "~" H 5900 3200 50  0001 C CNN
 	1    5900 3200
@@
 $EndComp
 $Comp
-L device:R R6
+L device:R R7
 U 1 1 5DBFE57D
 P 6700 3400
-F 0 "R6" H 6770 3446 50  0000 L CNN
+F 0 "R7" H 6770 3446 50  0000 L CNN
 F 1 "1k" H 6770 3355 50  0000 L CNN
-F 2 "Resistor_SMD:R_0603_1608Metric" V 6630 3400 50  0001 C CNN
+F 2 "Resistor_THT:R_Axial_DIN0207_L6.3mm_D2.5mm_P10.16mm_Horizontal" V 6630 3400 50  0001 C CNN
 F 3 "~" H 6700 3400 50  0001 C CNN
 	1    6700 3400
@@
 F 0 "SW1" H 4000 3935 50  0000 C CNN
 F 1 "SW_Push" H 4000 3844 50  0000 C CNN
-F 2 "Button_Switch_SMD:SW_SPST_B3S-1000" H 4000 3850 50  0001 C CNN
+F 2 "Button_Switch_THT:SW_PUSH_6mm_H4.3mm" H 4000 3850 50  0001 C CNN
 F 3 "" H 4000 3850 50  0001 C CNN
 	1    4000 3650
@@
 $EndComp
 $Comp
-L power:GND #PWR012
+L power:GND #PWR033
 U 1 1 5DC0092C
 P 4350 4550
-F 0 "#PWR012" H 4350 4300 50  0001 C CNN
+F 0 "#PWR033" H 4350 4300 50  0001 C CNN
 F 1 "GND" H 4355 4377 50  0000 C CNN
 F 2 "" H 4350 4550 50  0001 C CNN
@@
 $EndComp
 $Comp
-L power:GND #PWR010
+L power:GND #PWR031
 U 1 1 5DC0127C
 P 3700 4550
-F 0 "#PWR010" H 3700 4300 50  0001 C CNN
+F 0 "#PWR031" H 3700 4300 50  0001 C CNN
 F 1 "GND" H 3705 4377 50  0000 C CNN
 F 2 "" H 3700 4550 50  0001 C CNN
@@
 $EndComp
 $Comp
-L power:GND #PWR017
+L power:GND #PWR038
 U 1 1 5DC01C81
 P 5900 4550
-F 0 "#PWR017" H 5900 4300 50  0001 C CNN
+F 0 "#PWR038" H 5900 4300 50  0001 C CNN
 F 1 "GND" H 5905 4377 50  0000 C CNN
 F 2 "" H 5900 4550 50  0001 C CNN
@@
 	4350 3650 4800 3650
 $Comp
-L power:+5V #PWR011
+L power:+5V #PWR032
 U 1 1 5DC03078
 P 4350 2950
-F 0 "#PWR011" H 4350 2800 50  0001 C CNN
+F 0 "#PWR032" H 4350 2800 50  0001 C CNN
 F 1 "+5V" H 4365 3123 50  0000 C CNN
 F 2 "" H 4350 2950 50  0001 C CNN
@@
 $EndComp
 $Comp
-L power:+5V #PWR016
+L power:+5V #PWR037
 U 1 1 5DC045DB
 P 5900 2950
-F 0 "#PWR016" H 5900 2800 50  0001 C CNN
+F 0 "#PWR037" H 5900 2800 50  0001 C CNN
 F 1 "+5V" H 5915 3123 50  0000 C CNN
 F 2 "" H 5900 2950 50  0001 C CNN
@@
 $EndComp
 $Comp
-L power:+5V #PWR018
+L power:+5V #PWR039
 U 1 1 5DC04DD1
 P 6700 2950
-F 0 "#PWR018" H 6700 2800 50  0001 C CNN
+F 0 "#PWR039" H 6700 2800 50  0001 C CNN
 F 1 "+5V" H 6715 3123 50  0000 C CNN
 F 2 "" H 6700 2950 50  0001 C CNN
@@
 	5900 4450 5900 4550
 $Comp
-L power:GND #PWR013
+L power:GND #PWR034
 U 1 1 5DC08302
 P 5300 4550
-F 0 "#PWR013" H 5300 4300 50  0001 C CNN
+F 0 "#PWR034" H 5300 4300 50  0001 C CNN
 F 1 "GND" H 5305 4377 50  0000 C CNN
 F 2 "" H 5300 4550 50  0001 C CNN
@@
 Wire Wire Line
 	4350 3300 4350 2950
+$Comp
+L Connector_Generic:Conn_01x02 J4
+U 1 1 5DD07BEE
+P 4050 4050
+F 0 "J4" V 3922 4130 50  0000 L CNN
+F 1 "Conn_01x02" V 4013 4130 50  0000 L CNN
+F 2 "Connector_PinHeader_2.54mm:PinHeader_1x02_P2.54mm_Vertical" H 4050 4050 50  0001 C CNN
+F 3 "~" H 4050 4050 50  0001 C CNN
+	1    4050 4050
+	0    1    1    0
+$EndComp
+Wire Wire Line
+	4050 3850 4200 3850
+Wire Wire Line
+	4200 3850 4200 3650
+Connection ~ 4200 3650
+Wire Wire Line
+	3950 3850 3800 3850
+Wire Wire Line
+	3800 3850 3800 3650
+Connection ~ 3800 3650
 $EndSCHEMATC
